File: W2I-S100.kicad_sch (KiCad schematic)
At the start: 219 parts, among them J1 to WDI, J2 44-pin IDE, J3 Serial, J4 40-pin IDE, J5 EXT PWR, J6 Jumper to enable buzzer, P1 S100_MALE, P7 5V Reg, Q1 2N2222AU, SW1 SW_DIP_x07, U1 Z80CPU, U10 74HCT240, U101 74HCT138, U102 74LS123, U103 74LS123, U104 74HCT00, U11 74HCT374, U13 74HCT244, U14 74F138, U15 74HCT138, U16 74F138, U17 7438, U18 7438, U19 7438, U2 28C256, U20 7438, U21 74LS123, U22 74LS123, U23 74HCT165, U24 74HCT374, U25 74HCT164, U26 74F163, U27 74HCT393, U28 74HCT74, U29 74HCT138, U3 CY62256NLL-55ZXIT, U30 74HCT74, U31 74HCT374, U32 74HCT244, U33 74HCT244, U34 74HCT374, U35 74HCT374, U36 75107, U37 75110, U38 74HCT04, U39 74F04, U4 2681, U40 74F00, U41 74F08, U42 74F08, U43 74HCT32, U44 74HCT04, U45 74HCT14, U46 74HCT163, U47 74HCT02, U48 7905, U5 MAX232A, U50 3.3V LDO Reg, U6 74F74, U7 74F74, U8 74HCT374, U9 74LS244

Commit message: routing complete
Parts:
- added TP14: GND, TestPoint:TestPoint_THTPad_2.0x2.0mm_Drill1.0mm, symbol Connector:TestPoint
Connections:
- net GND: now also TP14.1
- net +8V: now reaches C70.1, J5.1 (Pin_1), P1.1 (+8_V), P1.51 (+8_V), P7.3 (VIN), TP10.1
- net +16V: now reaches P1.2 (+16_V), TP12.1
- net -16V: now reaches C72.2, J5.2 (Pin_2), P1.52 (-16_V), TP13.1, U48.2 (IN)
Other:
- moved on the sheet: TP12
Changed lines of the file:
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@@
 	)
 	(junction
+		(at 796.29 140.97)
+		(diameter 0)
+		(color 0 0 0 0)
+	)
+	(junction
 		(at 535.94 326.39)
 		(diameter 0)
@@
 	(wire
 		(pts
+			(xy 796.29 140.97) (xy 800.1 140.97)
+		)
+		(stroke
+			(width 0)
+			(type default)
+		)
+	)
+	(wire
+		(pts
 			(xy 763.27 391.16) (xy 763.27 388.62)
 		)
@@
 		)
 	)
+	(wire
+		(pts
+			(xy 796.29 140.97) (xy 796.29 157.48)
+		)
+		(stroke
+			(width 0)
+			(type default)
+		)
+	)
 	(bus
 		(pts
@@
 	(wire
 		(pts
+			(xy 796.29 157.48) (xy 787.4 157.48)
+		)
+		(stroke
+			(width 0)
+			(type default)
+		)
+	)
+	(wire
+		(pts
 			(xy 184.15 351.79) (xy 95.25 351.79)
 		)
@@
 	(wire
 		(pts
-			(xy 791.21 140.97) (xy 800.1 140.97)
+			(xy 791.21 140.97) (xy 796.29 140.97)
 		)
 		(stroke
@@
 	(wire
 		(pts
+			(xy 795.02 19.05) (xy 800.1 19.05)
+		)
+		(stroke
+			(width 0)
+			(type default)
+		)
+	)
+	(wire
+		(pts
 			(xy 542.29 34.29) (xy 542.29 39.37)
 		)
@@
 		)
 	)
+	(label "+16V"
+		(at 795.02 19.05 0)
+		(effects
+			(font
+				(size 1.27 1.27)
+			)
+			(justify left bottom)
+		)
+	)
 	(label "DataBus2"
 		(at 436.88 43.18 90)
@@
 		)
 	)
+	(label "-16V"
+		(at 767.08 129.54 0)
+		(effects
+			(font
+				(size 1.27 1.27)
+			)
+			(justify left bottom)
+		)
+	)
 	(label "DataBus7"
 		(at 252.73 292.1 0)
@@
 		)
 	)
+	(label "+8V"
+		(at 784.86 16.51 0)
+		(effects
+			(font
+				(size 1.27 1.27)
+			)
+			(justify left bottom)
+		)
+	)
 	(label "AddressBus6"
 		(at 326.39 92.71 0)
@@
 	)
 	(symbol
+		(lib_id "Connector:TestPoint")
+		(at 787.4 157.48 180)
+		(unit 1)
+		(exclude_from_sim no)
+		(in_bom yes)
+		(on_board yes)
+		(dnp no)
+		(fields_autoplaced yes)
+		(property "Reference" "TP14"
+			(at 789.94 159.5119 0)
+			(effects
+				(font
+					(size 1.27 1.27)
+				)
+				(justify right)
+			)
+		)
+		(property "Value" "GND"
+			(at 789.94 162.0519 0)
+			(effects
+				(font
+					(size 1.27 1.27)
+				)
+				(justify right)
+			)
+		)
+		(property "Footprint" "TestPoint:TestPoint_THTPad_2.0x2.0mm_Drill1.0mm"
+			(at 782.32 157.48 0)
+			(effects
+				(font
+					(size 1.27 1.27)
+				)
+				(hide yes)
+			)
+		)
+		(property "Datasheet" "~"
+			(at 782.32 157.48 0)
+			(effects
+				(font
+					(size 1.27 1.27)
+				)
+				(hide yes)
+			)
+		)
+		(property "Description" "test point"
+			(at 787.4 157.48 0)
+			(effects
+				(font
+					(size 1.27 1.27)
+				)
+				(hide yes)
+			)
+		)
+		(pin "1"
+		)
+		(instances
+			(project "W2I-S100"
+				(path "/461ad1b3-df41-4c8f-89ba-1a25d4188f9a"
+					(reference "TP14")
+					(unit 1)
+				)
+			)
+		)
+	)
+	(symbol
 		(lib_id "Device:R_US")
 		(at 166.37 368.3 270)
@@
 	(symbol
 		(lib_id "Connector:TestPoint")
-		(at 800.1 19.05 90)
+		(at 795.02 19.05 90)
 		(unit 1)
 		(exclude_from_sim no)
@@
 		(dnp no)
 		(property "Reference" "TP12"
-			(at 792.734 18.796 90)
+			(at 787.654 18.796 90)
 			(effects
 				(font
@@
 		)
 		(property "Value" "+16V"
-			(at 792.734 21.336 90)
+			(at 787.654 21.336 90)
 			(effects
 				(font
@@
 		)
 		(property "Footprint" "TestPoint:TestPoint_THTPad_2.0x2.0mm_Drill1.0mm"
-			(at 800.1 13.97 0)
+			(at 795.02 13.97 0)
 			(effects
 				(font
@@
 		)
 		(property "Datasheet" "~"
-			(at 800.1 13.97 0)
+			(at 795.02 13.97 0)
 			(effects
 				(font
@@
 		)
 		(property "Description" "test point"
-			(at 800.1 19.05 0)
+			(at 795.02 19.05 0)
 			(effects
 				(font

Commit message: part replacement & autorouter complete
Parts:
- U23: LCSC Part C456131 -> C352828
- U25: footprint footprints:TSSOP-14_L5.0-W4.4-P0.65-LS6.4-BL -> footprints:SOIC-14_L8.7-W3.9-P1.27-LS6.0-BL; LCSC Part C2908835 -> C547397
- U28, U30: LCSC Part C686657 -> C352961
- U43: footprint footprints:TSSOP-14_L5.0-W4.4-P0.65-LS6.4-BL -> footprints:SOIC-14_L8.7-W3.9-P1.27-LS6.0-BL; LCSC Part C547595 -> C6781
- U45: footprint footprints:TSSOP-14_L5.0-W4.4-P0.65-LS6.4-BL -> footprints:SOIC-14_L8.7-W3.9-P1.27-LS6.0-BL; LCSC Part C5968 -> C6769
Changed lines of the file:
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@@
 			)
 		)
-		(property "LCSC Part" "C686657"
+		(property "LCSC Part" "C352961"
 			(at 504.19 467.36 0)
 			(effects
@@
 			)
 		)
-		(property "LCSC Part" "C686657"
+		(property "LCSC Part" "C352961"
 			(at 388.62 474.98 0)
 			(effects
@@
 			)
 		)
-		(property "Footprint" "footprints:TSSOP-14_L5.0-W4.4-P0.65-LS6.4-BL"
+		(property "Footprint" "footprints:SOIC-14_L8.7-W3.9-P1.27-LS6.0-BL"
 			(at 392.43 144.78 0)
 			(effects
@@
 			)
 		)
-		(property "LCSC Part" "C5968"
+		(property "LCSC Part" "C6769"
 			(at 392.43 144.78 0)
 			(effects
@@
 			)
 		)
-		(property "Footprint" "footprints:TSSOP-14_L5.0-W4.4-P0.65-LS6.4-BL"
+		(property "Footprint" "footprints:SOIC-14_L8.7-W3.9-P1.27-LS6.0-BL"
 			(at 377.19 127 0)
 			(effects
@@
 			)
 		)
-		(property "LCSC Part" "C5968"
+		(property "LCSC Part" "C6769"
 			(at 377.19 127 0)
 			(effects
@@
 			)
 		)
-		(property "LCSC Part" "C686657"
+		(property "LCSC Part" "C352961"
 			(at 276.86 38.1 0)
 			(effects
@@
 			)
 		)
-		(property "Footprint" "footprints:TSSOP-14_L5.0-W4.4-P0.65-LS6.4-BL"
+		(property "Footprint" "footprints:SOIC-14_L8.7-W3.9-P1.27-LS6.0-BL"
 			(at 558.8 328.93 0)
 			(effects
@@
 			)
 		)
-		(property "LCSC Part" "C547595"
+		(property "LCSC Part" "C6781"
 			(at 558.8 328.93 0)
 			(effects
@@
 			)
 		)
-		(property "Footprint" "footprints:TSSOP-14_L5.0-W4.4-P0.65-LS6.4-BL"
+		(property "Footprint" "footprints:SOIC-14_L8.7-W3.9-P1.27-LS6.0-BL"
 			(at 292.1 187.96 0)
 			(effects
@@
 			)
 		)
-		(property "LCSC Part" "C5968"
+		(property "LCSC Part" "C6769"
 			(at 292.1 187.96 0)
 			(effects
@@
 			)
 		)
-		(property "LCSC Part" "C686657"
+		(property "LCSC Part" "C352961"
 			(at 411.48 127 0)
 			(effects
@@
 			)
 		)
-		(property "Footprint" "footprints:TSSOP-14_L5.0-W4.4-P0.65-LS6.4-BL"
+		(property "Footprint" "footprints:SOIC-14_L8.7-W3.9-P1.27-LS6.0-BL"
 			(at 646.43 467.36 0)
 			(effects
@@
 			)
 		)
-		(property "LCSC Part" "C547595"
+		(property "LCSC Part" "C6781"
 			(at 646.43 467.36 0)
 			(effects
@@
 			)
 		)
-		(property "Footprint" "footprints:TSSOP-14_L5.0-W4.4-P0.65-LS6.4-BL"
+		(property "Footprint" "footprints:SOIC-14_L8.7-W3.9-P1.27-LS6.0-BL"
 			(at 392.43 127 0)
 			(effects
@@
 			)
 		)
-		(property "LCSC Part" "C5968"
+		(property "LCSC Part" "C6769"
 			(at 392.43 127 0)
 			(effects
@@
 			)
 		)
-		(property "LCSC Part" "C456131"
+		(property "LCSC Part" "C352828"
 			(at 381 55.88 90)
 			(effects
@@
 			)
 		)
-		(property "Footprint" "footprints:TSSOP-14_L5.0-W4.4-P0.65-LS6.4-BL"
+		(property "Footprint" "footprints:SOIC-14_L8.7-W3.9-P1.27-LS6.0-BL"
 			(at 521.97 311.15 0)
 			(effects
@@
 			)
 		)
-		(property "LCSC Part" "C547595"
+		(property "LCSC Part" "C6781"
 			(at 521.97 311.15 0)
 			(effects
@@
 			)
 		)
-		(property "LCSC Part" "C686657"
+		(property "LCSC Part" "C352961"
 			(at 524.51 467.36 0)
 			(effects
@@
 			)
 		)
-		(property "Footprint" "footprints:TSSOP-14_L5.0-W4.4-P0.65-LS6.4-BL"
+		(property "Footprint" "footprints:SOIC-14_L8.7-W3.9-P1.27-LS6.0-BL"
 			(at 485.14 220.98 0)
 			(effects
@@
 			)
 		)
-		(property "LCSC Part" "C5968"
+		(property "LCSC Part" "C6769"
 			(at 485.14 220.98 90)
 			(effects
@@
 			)
 		)
-		(property "Footprint" "footprints:TSSOP-14_L5.0-W4.4-P0.65-LS6.4-BL"
+		(property "Footprint" "footprints:SOIC-14_L8.7-W3.9-P1.27-LS6.0-BL"
 			(at 312.42 187.96 0)
 			(effects
@@
 			)
 		)
-		(property "LCSC Part" "C5968"
+		(property "LCSC Part" "C6769"
 			(at 312.42 187.96 0)
 			(effects
@@
 			)
 		)
-		(property "LCSC Part" "C686657"
+		(property "LCSC Part" "C352961"
 			(at 541.02 276.86 0)
 			(effects
@@
 			)
 		)
-		(property "Footprint" "footprints:TSSOP-14_L5.0-W4.4-P0.65-LS6.4-BL"
+		(property "Footprint" "footprints:SOIC-14_L8.7-W3.9-P1.27-LS6.0-BL"
 			(at 523.24 328.93 0)
 			(effects
@@
 			)
 		)
-		(property "LCSC Part" "C547595"
+		(property "LCSC Part" "C6781"
 			(at 523.24 328.93 0)
 			(effects
@@
 			)
 		)
-		(property "Footprint" "footprints:TSSOP-14_L5.0-W4.4-P0.65-LS6.4-BL"
+		(property "Footprint" "footprints:SOIC-14_L8.7-W3.9-P1.27-LS6.0-BL"
 			(at 576.58 276.86 0)
 			(effects
@@
 			)
 		)
-		(property "LCSC Part" "C547595"
+		(property "LCSC Part" "C6781"
 			(at 576.58 276.86 0)
 			(effects
@@
 			)
 		)
-		(property "Footprint" "footprints:TSSOP-14_L5.0-W4.4-P0.65-LS6.4-BL"
+		(property "Footprint" "footprints:SOIC-14_L8.7-W3.9-P1.27-LS6.0-BL"
 			(at 687.07 467.36 0)
 			(effects
@@
 			)
 		)
-		(property "LCSC Part" "C5968"
+		(property "LCSC Part" "C6769"
 			(at 687.07 467.36 0)
 			(effects
@@
 			)
 		)
-		(property "Footprint" "footprints:TSSOP-14_L5.0-W4.4-P0.65-LS6.4-BL"
+		(property "Footprint" "footprints:SOIC-14_L8.7-W3.9-P1.27-LS6.0-BL"
 			(at 449.58 63.5 0)
 			(effects
@@
 			)
 		)
-		(property "LCSC Part" "C2908835"
+		(property "LCSC Part" "C547397"
 			(at 441.96 86.36 90)
 			(effects

Commit message: 3/28 updates
swapped crystals for TH parts
Parts:
- removed OSC1: 3.6864MHz, footprints:OSC-SMD_4P-L7.0-W5.0-BL-2, symbol easyeda2kicad:CB3-3C-3M686400
- removed OSC2: 27MHz, footprints:OSC-SMD_4P-L7.0-W5.0-BL-2, symbol easyeda2kicad:CB3-3C-27M000000
- added J7: Conn_01x02_Pin, Connector_PinHeader_2.54mm:PinHeader_1x02_P2.54mm_Vertical, symbol Connector:Conn_01x02_Pin
- added OSC1: ECS-2100AX-3.6864MHZ, Oscillator:Oscillator_DIP-8, symbol Oscillator:CXO_DIP8
- added OSC2: ACHL-27.000MHZ-EK, Oscillator:Oscillator_DIP-8, symbol Oscillator:CXO_DIP8
- added R16: 22K, footprints:R1206, symbol Device:R_US
- added R17: 4.7K, footprints:R1206, symbol Device:R_US
Connections:
- net +5V: now also C10.2, C11.2, OSC1.1 (EN), OSC1.8 (Vcc), OSC2.1 (EN), OSC2.8 (Vcc), R16.2, R17.1; no longer C10.1, C11.1, U9.13 (I1b)
- net GND: now also C10.1, C11.1, J7.1 (Pin_1), OSC1.4 (GND), OSC2.4 (GND); no longer C10.2, C11.2
- net IDEDataBus7: now also R16.1
- net at U28.11 (C): now also OSC2.5 (OUT)
- net at U4.20 (X1): now also OSC1.5 (OUT)
- new net: J7.2 (Pin_2), R17.2, U9.13 (I1b)
Other:
- moved on the sheet: C10, C11

Commit message: W2I-S100 Rev 1 Final
Parts:
- added TP15: U8-16, TestPoint:TestPoint_THTPad_2.0x2.0mm_Drill1.0mm, symbol Connector:TestPoint
- BZ1: value Buzzer -> PKHPS0013E4000-A2
- R10: value 100 -> 330
- RP1: value 761-5-R220/330 -> 4116R-3-221/331
- U1: value Z80CPU -> Z84C0020PEC
Connections:
- net at U8.16 (O6): now also TP15.1
- no-connect marks 35 -> 34
Other:
- note added: "(min 180R)"
Changed lines of the file:
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@@
 		)
 	)
+	(text "(min 180R)"
+		(exclude_from_sim no)
+		(at 547.116 157.48 0)
+		(effects
+			(font
+				(size 1.27 1.27)
+			)
+		)
+	)
 	(junction
 		(at 494.03 233.68)
@@
 	)
 	(junction
+		(at 176.53 299.72)
+		(diameter 0)
+		(color 0 0 0 0)
+	)
+	(junction
 		(at 784.86 64.77)
 		(diameter 0)
@@
 	)
 	(junction
-		(at 180.34 299.72)
-		(diameter 0)
-		(color 0 0 0 0)
-	)
-	(junction
 		(at 457.2 86.36)
 		(diameter 0)
@@
 	)
 	(no_connect
-		(at 184.15 297.18)
-	)
-	(no_connect
 		(at 129.54 102.87)
 	)
@@
 	(wire
 		(pts
+			(xy 182.88 297.18) (xy 184.15 297.18)
+		)
+		(stroke
+			(width 0)
+			(type default)
+		)
+	)
+	(wire
+		(pts
 			(xy 496.57 134.62) (xy 501.65 134.62)
 		)
@@
 	(wire
 		(pts
-			(xy 180.34 299.72) (xy 184.15 299.72)
-		)
-		(stroke
-			(width 0)
-			(type default)
-		)
-	)
-	(wire
-		(pts
 			(xy 594.36 454.66) (xy 594.36 464.82)
 		)
@@
 	(wire
 		(pts
-			(xy 170.18 299.72) (xy 180.34 299.72)
+			(xy 170.18 299.72) (xy 176.53 299.72)
 		)
 		(stroke
@@
 		)
 	)
+	(wire
+		(pts
+			(xy 176.53 299.72) (xy 184.15 299.72)
+		)
+		(stroke
+			(width 0)
+			(type default)
+		)
+	)
 	(bus
 		(pts
@@
 	(wire
 		(pts
+			(xy 182.88 264.16) (xy 182.88 297.18)
+		)
+		(stroke
+			(width 0)
+			(type default)
+		)
+	)
+	(wire
+		(pts
 			(xy 208.28 210.82) (xy 283.21 210.82)
 		)
@@
 	(wire
 		(pts
-			(xy 180.34 307.34) (xy 180.34 299.72)
+			(xy 176.53 307.34) (xy 176.53 299.72)
 		)
 		(stroke
@@
 	)
 	(label "+FAULT"
-		(at 180.34 307.34 90)
+		(at 176.53 307.34 90)
 		(effects
 			(font
@@
 			)
 		)
-		(property "Value" "Z80CPU"
+		(property "Value" "Z84C0020PEC"
 			(at 310.7533 71.12 0)
 			(effects
@@
 	)
 	(symbol
+		(lib_id "Connector:TestPoint")
+		(at 182.88 264.16 0)
+		(unit 1)
+		(exclude_from_sim no)
+		(in_bom yes)
+		(on_board yes)
+		(dnp no)
+		(fields_autoplaced yes)
+		(property "Reference" "TP15"
+			(at 185.42 259.5879 0)
+			(effects
+				(font
+					(size 1.27 1.27)
+				)
+				(justify left)
+			)
+		)
+		(property "Value" "U8-16"
+			(at 185.42 262.1279 0)
+			(effects
+				(font
+					(size 1.27 1.27)
+				)
+				(justify left)
+			)
+		)
+		(property "Footprint" "TestPoint:TestPoint_THTPad_2.0x2.0mm_Drill1.0mm"
+			(at 187.96 264.16 0)
+			(effects
+				(font
+					(size 1.27 1.27)
+				)
+				(hide yes)
+			)
+		)
+		(property "Datasheet" "~"
+			(at 187.96 264.16 0)
+			(effects
+				(font
+					(size 1.27 1.27)
+				)
+				(hide yes)
+			)
+		)
+		(property "Description" "test point"
+			(at 182.88 264.16 0)
+			(effects
+				(font
+					(size 1.27 1.27)
+				)
+				(hide yes)
+			)
+		)
+		(pin "1"
+		)
+		(instances
+			(project "W2I-S100"
+				(path "/461ad1b3-df41-4c8f-89ba-1a25d4188f9a"
+					(reference "TP15")
+					(unit 1)
+				)
+			)
+		)
+	)
+	(symbol
 		(lib_id "Connector_Generic:Conn_02x12_Counter_Clockwise")
 		(at 115.57 87.63 0)
@@
 			)
 		)
-		(property "Value" "761-5-R220/330"
+		(property "Value" "4116R-3-221/331"
 			(at 84.582 450.85 90)
 			(effects
@@
 		(on_board yes)
 		(dnp no)
-		(fields_autoplaced yes)
 		(property "Reference" "R10"
 			(at 560.07 148.5899 0)
@@
 			)
 		)
-		(property "Value" "100"
+		(property "Value" "330"
 			(at 560.07 151.1299 0)
 			(effects
@@
 			)
 		)
-		(property "Value" "Buzzer"
+		(property "Value" "PKHPS0013E4000-A2"
 			(at 564.642 159.258 90)
 			(effects
@@
 			)
 		)
-		(property "Description" "Buzzer, polarized"
+		(property "Description" ""
 			(at 565.15 154.94 0)
 			(effects
